Commit message: update cobot usd

File: asset/robot/urdf/cobot.urdf (robot description, URDF)
Before this commit: robot cobot, 14 links, 13 joints
Links:
- added link grasp_target, mass 0.0; visual box size=0.02 0.02 0.02
- link base: mass None -> 0.8; geometry collision mesh filename=meshes/base.stl; visual mesh filename=meshes/base.stl
- link link1: mass 2.34 -> 0.5; geometry collision mesh filename=meshes/link1.stl; visual mesh filename=meshes/link1.stl
- link link2: mass 2.34 -> 0.5; geometry collision mesh filename=meshes/link2.stl; visual mesh filename=meshes/link2.stl
- link link3: mass 2.34 -> 0.4; geometry collision mesh filename=meshes/link3.stl; visual mesh filename=meshes/link3.stl
- link link4: mass 2.34 -> 0.3; geometry collision mesh filename=meshes/link4.stl; visual mesh filename=meshes/link4.stl
- link link5: mass 2.34 -> 0.2; geometry collision mesh filename=meshes/link5.stl; visual mesh filename=meshes/link5.stl
- link link6: mass None -> 0.1
Joints:
- removed joint base_to_left1
- removed joint base_to_link1
- removed joint link1_to_link2
- removed joint link2_to_link3
- removed joint link3_to_link4
- removed joint link4_to_link5
- removed joint link5_to_link6
- added joint cobot_joint1: type revolute, parent base, child link1, origin xyz=0 0 0.162 rpy=0 0 0, axis 0 0 1, limit lower=-2.96 upper=2.96 effort=1000.0 velocity=0
- added joint cobot_joint2: type revolute, parent link1, child link2, origin xyz=0 0 0 rpy=0 -1.5708 1.5708, axis 0 0 1, limit lower=-2.79 upper=2.79 effort=1000.0 velocity=0
- added joint cobot_joint3: type revolute, parent link2, child link3, origin xyz=0.13635 0 0 rpy=0 0 0 , axis 0 0 1, limit lower=-2.79 upper=2.79 effort=1000.0 velocity=0
- added joint cobot_joint4: type revolute, parent link3, child link4, origin xyz=0.1205 0 0.082 rpy=0 0 1.57080 , axis 0 0 1, limit lower=-2.79 upper=2.79 effort=1000.0 velocity=0
- added joint cobot_joint5: type revolute, parent link4, child link5, origin xyz=0 -0.084 0.0 rpy=1.5708 0 0, axis 0 0 1, limit lower=-2.96 upper=2.96 effort=1000.0 velocity=0
- added joint cobot_joint6: type revolute, parent link5, child link6, origin xyz=0 0.06635 0.0 rpy=-1.5708 0 0, axis 0 0 1, limit lower=-3.05 upper=3.05 effort=1000.0 velocity=0
- added joint grasptarget_hand: type fixed, parent gripper_base, child grasp_target, origin xyz=0.14 0 -0.016 rpy=0 0 0
- added joint gripper_controller: type revolute, parent gripper_base, child gripper_left_link1, origin xyz=0.028185 0.044392 -0.0189 rpy=0 0 0.00017976, axis 0 0 1, limit lower=-1.57 upper=1.57 effort=100 velocity=10
- joint base_to_left3: mimic joint=base_to_left1 multiplier=1 offset=0 -> joint=gripper_controller multiplier=1 offset=0
- joint base_to_right1: mimic joint=base_to_left1 multiplier=-1 offset=0 -> joint=gripper_controller multiplier=-1 offset=0
- joint left1_to_left2: mimic joint=base_to_left1 multiplier=-1 offset=0 -> joint=gripper_controller multiplier=-1 offset=0
- joint robot_to_hand: limit lower=-3.05 upper=3.05 effort=1000.0 velocity=0 -> lower=-3.05 upper=3.05 effort=100.0 velocity=0
